Commit message: changed model orientation

File: robot/description/robot.urdf.xacro (robot description, xacro)
@@ -2,3 +2,4 @@
 <robot xmlns:xacro="http://www.ros.org/wiki/xacro" name="robot">
     <xacro:include filename="robot_core.xacro" />
+    <xacro:include filename="gazebo_control.xacro"/>
 </robot>

File: robot/description/robot_core.xacro (robot description, xacro)
@@ -26,5 +26,5 @@
     <link name="chassis">
         <visual>
-            <origin xyz="0.15 0 0.25" rpy="0 0 0" />
+            <origin xyz="0.05 0 0.25" rpy="0 0 0" />
             <geometry>
                 <cylinder length="0.5" radius="0.165" />
@@ -33,5 +33,5 @@
         </visual>
         <collision>
-            <origin xyz="0.15 0 0.25" rpy="0 0 0" />
+            <origin xyz="0.05 0 0.25" rpy="0 0 0" />
             <geometry>
                 <cylinder length="0.5" radius="0.165" />
@@ -42,4 +42,7 @@
         </xacro:inertial_box>
     </link>
+    <gazebo reference="chassis">
+        <material>Gazebo/White</material>
+    </gazebo>
     <!-- LEFT WHEEL -->
     <joint name="left_wheel_joint" type="continuous">
@@ -66,9 +69,12 @@
         </xacro:inertial_cylinder>
     </link>
+    <gazebo reference="left_wheel">
+        <material>Gazebo/Blue</material>
+    </gazebo>
     <!-- RIGHT WHEEL -->
     <joint name="right_wheel_joint" type="continuous">
         <parent link="base_link" />
         <child link="right_wheel" />
-        <origin xyz="0 -0.185 0" rpy="${pi/2} 0 0" />
+s        <origin xyz="0 -0.185 0" rpy="${pi/2} 0 0" />
         <axis xyz="0 0 -1" />
     </joint>
@@ -90,9 +96,12 @@
         </xacro:inertial_sphere>
     </link>
+    <gazebo reference="right_wheel">
+        <material>Gazebo/Blue</material>
+    </gazebo>
     <!-- CASTER WHEEL -->
     <joint name="caster_wheel_joint" type="fixed">
         <parent link="chassis" />
         <child link="caster_wheel" />
-        <origin xyz="0.24 0 0" rpy="0 0 0" />
+        <origin xyz="-0.05 0 0" rpy="0 0 0" />
     </joint>
     <link name="caster_wheel">
@@ -110,3 +119,8 @@
         </collision>
     </link>
+    <gazebo reference="caster_wheel">
+        <material>Gazebo/Black</material>
+        <mu1 value="0.001"/>
+        <mu2 value="0.001"/>
+    </gazebo>
 </robot>
