Commit message: changed urdf model

File: src/sam_bot_description/src/description/sam_bot_description.urdf (robot description, URDF)
Before this commit: robot sam_bot, 7 links, 6 joints
Joints:
- joint caster_joint: origin xyz=${caster_xoff} 0.0 ${-(base_height/2)} rpy=0 0 0 -> xyz=-${caster_xoff} 0.0 ${-(base_height/2)} rpy=0 0 0
- joint lidar_joint: origin xyz=0 0 0.12 rpy=0 0 0 -> xyz=0 0 0.35 rpy=0 0 0

Commit message: changed urdf model

File: src/sam_bot_description/src/description/sam_bot_description.urdf (robot description, URDF)
Before this commit: robot sam_bot, 5 links, 4 joints
Links:
- removed link base_footprint
- removed link base_link
- removed link front_caster
- removed link imu_link
- removed link lidar_link
Joints:
- removed joint base_joint
- removed joint caster_joint
- removed joint imu_joint
- removed joint lidar_joint
