Commit message: hardware control done

File: src/robot_description/src/description/ros2_control.xacro (robot description, xacro)
@@ -5,25 +5,24 @@
             <plugin>gazebo_ros2_control/GazeboSystem</plugin>
         </hardware>
-        <joint name="drivewhl_l">
+        <joint name="drivewhl_l_joint">
             <command_interface name="velocity">
                 <param name="min">-10</param>
                 <param name="max">10</param>
             </command_interface>
-            <state_interface name="velocity" />
-            <state_interface name="position" />
+            <state_interface name="velocity"/>
+            <state_interface name="position"/>
         </joint>
-        <joint name="drivewhl_r">
+        <joint name="drivewhl_r_joint">
             <command_interface name="velocity">
                 <param name="min">-10</param>
                 <param name="max">10</param>
             </command_interface>
-            <state_interface name="velocity" />
-            <state_interface name="position" />
+            <state_interface name="velocity"/>
+            <state_interface name="position"/>
         </joint>
     </ros2_control>
     <gazebo>
-        <plugin name='gazebo_ros2_control' filename='libgazebo_ros2_control.so'>
-            <parameters
-            >$(find robot_description/config/my_controllers.yaml)</parameters>
+        <plugin name="gazebo_ros2_control" filename="libgazebo_ros2_control.so">
+        <parameters>$(find robot_description)/config/my_controllers.yaml</parameters>
         </plugin>
     </gazebo>
