Commit message: updated urdf

File: src/robot_description/src/description/robot_constants.xacro (robot description, xacro)
@@ -8,5 +8,5 @@
     <xacro:property name="wheel_ygap" value="0.025" />
     <xacro:property name="wheel_zoff" value="0.05" />
-    <xacro:property name="wheel_xoff" value="0.12" />
+    <xacro:property name="wheel_xoff" value="0.05" />
     <xacro:property name="caster_xoff" value="0.14" />
 </robot>
