Commit message: changed urdf model

File: src/robot_description/src/description/bot_core.xacro (robot description, xacro)
@@ -70,5 +70,5 @@
     <xacro:wheel prefix="drivewhl_l" x_reflect="1" y_reflect="1" />
     <xacro:wheel prefix="drivewhl_r" x_reflect="1" y_reflect="-1" />
-    <link name="front_caster">
+    <link name="back_caster">
         <visual>
         <geometry>
@@ -92,5 +92,5 @@
     <joint name="caster_joint" type="fixed">
         <parent link="base_link" />
-        <child link="front_caster" />
+        <child link="back_caster" />
         <origin xyz="-${caster_xoff} 0.0 ${-(base_height/2)}" rpy="0 0 0" />
     </joint>

File: src/robot_description/src/description/imu.xacro (robot description, xacro)
@@ -1,4 +1,5 @@
 <?xml version="1.0" ?>
 <robot xmlns:xacro="http://ros.org/wiki/xacro">
+    <xacro:include filename="inertial_macros.xacro" />
     <link name="imu_link">
         <visual>

Commit message: changed urdf visuals

File: src/robot_description/src/description/bot_core.xacro (robot description, xacro)
@@ -6,10 +6,11 @@
     <link name="base_link">
         <visual>
-        <geometry>
-            <box size="${base_length} ${base_width} ${base_height}" />
-        </geometry>
-        <material name="Cyan">
-            <color rgba="0 1.0 1.0 1.0" />
-        </material>
+            <geometry>
+                <!--<box size="${base_length} ${base_width} ${base_height}" />-->
+                <cylinder radius="${base_length/2}" length="${base_height}" />
+            </geometry>
+            <material name="orange">
+                <color rgba="1 0.3 0.1 1" />
+            </material>
         </visual>
         <collision>
@@ -25,4 +26,7 @@
         />
     </link>
+    <gazebo reference="base_link">
+        <material>Gazebo/Orange</material>
+    </gazebo>
     <!-- Robot Footprint -->
     <link name="base_footprint">
@@ -42,6 +46,6 @@
             <cylinder radius="${wheel_radius}" length="${wheel_width}" />
             </geometry>
-            <material name="Gray">
-            <color rgba="0.5 0.5 0.5 1.0" />
+            <material name="blue">
+                <color rgba="0.2 0.2 1 1" />
             </material>
         </visual>
@@ -70,12 +74,18 @@
     <xacro:wheel prefix="drivewhl_l" x_reflect="1" y_reflect="1" />
     <xacro:wheel prefix="drivewhl_r" x_reflect="1" y_reflect="-1" />
+    <gazebo reference="drivewhl_l_link">
+        <material>Gazebo/Blue</material>
+    </gazebo>
+    <gazebo reference="drivewhl_r_link">
+        <material>Gazebo/Blue</material>
+    </gazebo>
     <link name="back_caster">
         <visual>
-        <geometry>
-            <sphere radius="${(wheel_radius+wheel_zoff-(base_height/2))}" />
-        </geometry>
-        <material name="Cyan">
-            <color rgba="0 1.0 1.0 1.0" />
-        </material>
+            <geometry>
+                <sphere radius="${(wheel_radius+wheel_zoff-(base_height/2))}" />
+            </geometry>
+            <material name="blue">
+                <color rgba="0.2 0.2 1 1" />
+            </material>
         </visual>
         <collision>

File: src/robot_description/src/description/lidar.xacro (robot description, xacro)
@@ -3,19 +3,29 @@
     <link name="lidar_link">
         <inertial>
-        <origin xyz="0 0 0" rpy="0 0 0" />
-        <mass value="0.125" />
-        <inertia ixx="0.001" ixy="0" ixz="0" iyy="0.001" iyz="0" izz="0.001" />
+            <origin xyz="0 0 0" rpy="0 0 0" />
+            <mass value="0.125" />
+            <inertia
+                ixx="0.001"
+                ixy="0"
+                ixz="0"
+                iyy="0.001"
+                iyz="0"
+                izz="0.001"
+            />
         </inertial>
         <collision>
-        <origin xyz="0 0 0" rpy="0 0 0" />
-        <geometry>
-            <cylinder radius="0.0508" length="0.055" />
-        </geometry>
+            <origin xyz="0 0 0" rpy="0 0 0" />
+            <geometry>
+                <cylinder radius="0.0508" length="0.055" />
+            </geometry>
         </collision>
         <visual>
-        <origin xyz="0 0 0" rpy="0 0 0" />
-        <geometry>
-            <cylinder radius="0.0508" length="0.055" />
-        </geometry>
+            <origin xyz="0 0 0" rpy="0 0 0" />
+            <geometry>
+                <cylinder radius="0.0508" length="0.055" />
+            </geometry>
+            <material name="black">
+                <color rgba="0 0 0 1" />
+            </material>
         </visual>
     </link>
@@ -26,4 +36,5 @@
     </joint>
     <gazebo reference="lidar_link">
+        <material>Gazebo/Black</material>
         <sensor name="lidar" type="ray">
         <always_on>true</always_on>

Commit message: hardware controller done

File: src/robot_description/src/description/bot_core.xacro (robot description, xacro)
@@ -53,5 +53,5 @@
             <origin xyz="0 0 0" rpy="${pi/2} 0 0" />
             <geometry>
-            <cylinder radius="${wheel_radius}" length="${wheel_width}" />
+            <sphere radius="${wheel_radius}" />
             </geometry>
         </collision>

File: src/robot_description/src/description/lidar.xacro (robot description, xacro)
@@ -43,20 +43,20 @@
         <ray>
             <scan>
-            <horizontal>
-                <samples>360</samples>
-                <resolution>1.000000</resolution>
-                <min_angle>0.000000</min_angle>
-                <max_angle>6.280000</max_angle>
-            </horizontal>
+                <horizontal>
+                    <samples>360</samples>
+                    <resolution>1.000000</resolution>
+                    <min_angle>0.000000</min_angle>
+                    <max_angle>6.280000</max_angle>
+                </horizontal>
             </scan>
             <range>
-            <min>0.120000</min>
-            <max>3.5</max>
-            <resolution>0.015000</resolution>
+                <min>0.3</min>
+                <max>12</max>
+                <resolution>0.015000</resolution>
             </range>
             <noise>
-            <type>gaussian</type>
-            <mean>0.0</mean>
-            <stddev>0.01</stddev>
+                <type>gaussian</type>
+                <mean>0.0</mean>
+                <stddev>0.01</stddev>
             </noise>
         </ray>

File: src/robot_description/src/description/ros2_control.xacro (robot description, xacro)
@@ -1,25 +1,57 @@
 <?xml version="1.0" ?>
 <robot xmlns:xacro="http://ros.org/wiki/xacro">
-    <ros2_control name="GazeboSystem" type="system">
-        <hardware>
-            <plugin>gazebo_ros2_control/GazeboSystem</plugin>
-        </hardware>
-        <joint name="drivewhl_l_joint">
-            <command_interface name="velocity">
-                <param name="min">-10</param>
-                <param name="max">10</param>
-            </command_interface>
-            <state_interface name="velocity"/>
-            <state_interface name="position"/>
-        </joint>
-        <joint name="drivewhl_r_joint">
-            <command_interface name="velocity">
-                <param name="min">-10</param>
-                <param name="max">10</param>
-            </command_interface>
-            <state_interface name="velocity"/>
-            <state_interface name="position"/>
-        </joint>
-    </ros2_control>
+    <xacro:unless value="$(arg sim_mode)">
+        <ros2_control name="RealRobot" type="system">
+            <hardware>
+                <plugin>diffdrive_arduino/DiffDriveArduinoHardware</plugin>
+                <param name="right_wheel_name">drivewhl_r_joint</param>
+                <param name="left_wheel_name">drivewhl_l_joint</param>
+                <param name="loop_rate">30</param>
+                <param name="device">/dev/ttyUSB0</param>
+                <param name="baud_rate">57600</param>
+                <param name="timeout_ms">1000</param>
+                <param name="enc_counts_per_rev">3450</param>
+            </hardware>
+            <joint name="drivewhl_l_joint">
+                <command_interface name="velocity">
+                    <param name="min">-10</param>
+                    <param name="max">10</param>
+                </command_interface>
+                <state_interface name="position"/>
+                <state_interface name="velocity"/>
+            </joint>
+            <joint name="drivewhl_r_joint">
+                <command_interface name="velocity">
+                    <param name="min">-10</param>
+                    <param name="max">10</param>
+                </command_interface>
+                <state_interface name="position"/>
+                <state_interface name="velocity"/>
+            </joint>
+        </ros2_control>
+    </xacro:unless>
+    <xacro:if value="$(arg sim_mode)">
+        <ros2_control name="GazeboSystem" type="system">
+            <hardware>
+                <plugin>gazebo_ros2_control/GazeboSystem</plugin>
+            </hardware>
+            <joint name="drivewhl_l_joint">
+                <command_interface name="velocity">
+                    <param name="min">-10</param>
+                    <param name="max">10</param>
+                </command_interface>
+                <state_interface name="velocity"/>
+                <state_interface name="position"/>
+            </joint>
+            <joint name="drivewhl_r_joint">
+                <command_interface name="velocity">
+                    <param name="min">-10</param>
+                    <param name="max">10</param>
+                </command_interface>
+                <state_interface name="velocity"/>
+                <state_interface name="position"/>
+            </joint>
+        </ros2_control>
+    </xacro:if>
     <gazebo>
         <plugin name="gazebo_ros2_control" filename="libgazebo_ros2_control.so">

Commit message: uwb urdf

File: src/robot_description/src/description/bot_core.xacro (robot description, xacro)
@@ -16,5 +16,5 @@
         <collision>
         <geometry>
-            <box size="${base_length} ${base_width} ${base_height}" />
+            <box size="${base_length/1.25} ${base_width/1.25} ${base_height}" />
         </geometry>
         </collision>
