Commit message: changed urdf visuals

File: src/robot_description/src/description/lidar.xacro (robot description, xacro)
@@ -1,5 +1,5 @@
 <?xml version="1.0" ?>
 <robot xmlns:xacro="http://ros.org/wiki/xacro">
-    <link name="lidar_link">
+    <link name="laser_frame">
         <inertial>
             <origin xyz="0 0 0" rpy="0 0 0" />
@@ -30,10 +30,10 @@
         </visual>
     </link>
-    <joint name="lidar_joint" type="fixed">
+    <joint name="laser_joint" type="fixed">
         <parent link="base_link" />
-        <child link="lidar_link" />
+        <child link="laser_frame" />
         <origin xyz="0 0 0.35" rpy="0 0 0" />
     </joint>
-    <gazebo reference="lidar_link">
+    <gazebo reference="laser_frame">
         <material>Gazebo/Black</material>
         <sensor name="lidar" type="ray">
@@ -66,5 +66,5 @@
             </ros>
             <output_type>sensor_msgs/LaserScan</output_type>
-            <frame_name>lidar_link</frame_name>
+            <frame_name>laser_frame</frame_name>
         </plugin>
         </sensor>

Commit message: uwb urdf

File: src/robot_description/src/description/lidar.xacro (robot description, xacro)
@@ -33,5 +33,5 @@
         <parent link="base_link" />
         <child link="laser_frame" />
-        <origin xyz="0 0 0.35" rpy="0 0 0" />
+        <origin xyz="0 0 0.55" rpy="0 0 0" />
     </joint>
     <gazebo reference="laser_frame">

File: src/robot_description/src/description/uwb.xacro (robot description, xacro)
@@ -5,5 +5,5 @@
             <origin xyz="0 0 0" rpy="0 0 0" />
             <geometry>
-                <box size="0.05 0.02 0.02" />
+                <box size="0.05 0.05 0.05" />
             </geometry>
             <material name="">
@@ -15,5 +15,5 @@
         <parent link="base_link" />
         <child link="uwb_frame" />
-        <origin xyz="0 0 0.18" />
+        <origin xyz="0 0 0.20" />
     </joint>
 </robot>

Commit message: uwb urdf and lidar updated

File: src/robot_description/src/description/lidar.xacro (robot description, xacro)
@@ -1,4 +1,5 @@
 <?xml version="1.0" ?>
 <robot xmlns:xacro="http://ros.org/wiki/xacro">
+    <xacro:include filename="robot_constants.xacro"/>
     <link name="laser_frame">
         <inertial>
@@ -33,5 +34,5 @@
         <parent link="base_link" />
         <child link="laser_frame" />
-        <origin xyz="0 0 0.55" rpy="0 0 0" />
+        <origin xyz="-${base_width/2} 0 0.5" rpy="0 0 0" />
     </joint>
     <gazebo reference="laser_frame">

File: src/robot_description/src/description/uwb.xacro (robot description, xacro)
@@ -1,4 +1,5 @@
 <?xml version="1.0" ?>
 <robot xmlns:xacro="http://ros.org/wiki/xacro">
+    <xacro:include filename="robot_constants.xacro"/>
     <link name="uwb_frame">
         <visual>
@@ -8,5 +9,5 @@
             </geometry>
             <material name="">
-                <color rgba="0 0 0 0.24" />
+                <color rgba="1 1 1 1" />
             </material>
         </visual>
@@ -15,5 +16,5 @@
         <parent link="base_link" />
         <child link="uwb_frame" />
-        <origin xyz="0 0 0.20" />
+        <origin xyz="${base_width/2 - 0.05/2} 0 0.20" />
     </joint>
 </robot>
